Commit message: update amr_description

File: robot_ws/src/amr_description/urdf/actuator/caster.urdf.xacro (robot description, xacro)
@@ -1,7 +1,7 @@
 <?xml version="1.0"?>
 <robot xmlns:xacro="http://www.ros.org/wiki/xacro">
-    <xacro:include filename="$(find amr_description)/urdf/amr_description/common_inertia.xacro"/>
-    <xacro:macro name="caster_xacro" params="caster_name radius xyz">
-        <link name="${caster_name}_caster_link">
+    <xacro:include filename="$(find amr_description)/urdf/common_inertia.xacro"/>
+    <xacro:macro name="caster_xacro" params="caster_name radius xyz prefix">
+        <link name="${prefix}${caster_name}_caster_link">
             <visual>
                 <geometry>
@@ -20,10 +20,10 @@
             <xacro:sphere_inertia m="${1.5}" r="${radius}"/>
         </link>
-        <joint name="${caster_name}_caster_joint" type="continuous">
-            <parent link="base_link"/>
-            <child link="${caster_name}_caster_link"/>
+        <joint name="${prefix}${caster_name}_caster_joint" type="continuous">
+            <parent link="${prefix}base_link"/>
+            <child link="${prefix}${caster_name}_caster_link"/>
             <origin xyz="${xyz}"/>
         </joint>
-        <gazebo reference="${caster_name}_caster_link">
+        <gazebo reference="${prefix}${caster_name}_caster_link">
             <material>Gazebo/Yellow</material>
             <mu1 value="0.0"/>

File: robot_ws/src/amr_description/urdf/actuator/wheel.urdf.xacro (robot description, xacro)
@@ -1,7 +1,7 @@
 <?xml version="1.0"?>
 <robot xmlns:xacro="http://www.ros.org/wiki/xacro">
-    <xacro:include filename="$(find amr_description)/urdf/amr_description/common_inertia.xacro"/>
-    <xacro:macro name="wheel_xacro" params="wheel_name radius length xyz">
-        <link name="${wheel_name}_wheel_link">
+    <xacro:include filename="$(find amr_description)/urdf/common_inertia.xacro"/>
+    <xacro:macro name="wheel_xacro" params="wheel_name radius length xyz prefix mass">
+        <link name="${prefix}${wheel_name}_wheel_link">
             <visual>
                 <geometry>
@@ -18,13 +18,13 @@
                 <material name="yellow"/>
             </collision>
-            <xacro:cylinder_inertia m="${1.0}" r="${radius}" h="${length}"/>
+            <xacro:cylinder_inertia m="${mass}" r="${radius}" h="${length}"/>
         </link>
-        <joint name="${wheel_name}_wheel_joint" type="continuous">
-            <parent link="base_link"/>
-            <child link="${wheel_name}_wheel_link"/>
+        <joint name="${prefix}${wheel_name}_wheel_joint" type="continuous">
+            <parent link="${prefix}base_link"/>
+            <child link="${prefix}${wheel_name}_wheel_link"/>
             <origin xyz="${xyz}"/>
             <axis xyz="0 1 0"/>
         </joint>
-        <gazebo reference="${wheel_name}_wheel_link">
+        <gazebo reference="${prefix}${wheel_name}_wheel_link">
             <material>Gazebo/Yellow</material>
             <mu1 value="20.0"/>

File: robot_ws/src/amr_description/urdf/amr.ros2_control.xacro (robot description, xacro)
@@ -1,5 +1,12 @@
 <?xml version="1.0"?>
 <robot xmlns:xacro="http://www.ros.org/wiki/xacro">
-    <xacro:macro name="amr_ros2_control" params="left_joint_name right_joint_name">
+    <!--
+        left_joint_name / right_joint_name  带前缀的轮关节名
+        prefix            TF 帧前缀（如 robot01_），用于控制器 joint / 坐标系参数
+        namespace         controller_manager 的命名空间（如 robot01，空为根）
+        controller_params 控制器参数文件路径（默认 amr_ros2_controller.yaml 模板；
+                          生成脚本按机器人规格生成并传入）
+    -->
+    <xacro:macro name="amr_ros2_control" params="left_joint_name right_joint_name prefix namespace controller_params">
         <ros2_control name="AmrRobotGazeboSystem" type="system">
                 <hardware>
@@ -35,8 +42,9 @@
         <gazebo>
             <plugin filename="libgazebo_ros2_control.so" name="gazebo_ros2_control">
-                <parameters>$(find amr_description)/config/amr_ros2_controller.yaml</parameters>
+                <parameters>${controller_params}</parameters>
                 <ros>
-                    <remapping>/amr_diff_drive_controller/cmd_vel_unstamped:=/cmd_vel</remapping>
-                    <remapping>/amr_diff_drive_controller/odom:=/odom</remapping>
+                    <namespace>${namespace}</namespace>
+                    <remapping>amr_diff_drive_controller/cmd_vel_unstamped:=cmd_vel</remapping>
+                    <remapping>amr_diff_drive_controller/odom:=odom</remapping>
                 </ros>
             </plugin>

File: robot_ws/src/amr_description/urdf/amr.urdf.xacro (robot description, xacro)
@@ -1,27 +1,36 @@
 <?xml version="1.0"?>
 <robot xmlns:xacro="http://www.ros.org/wiki/xacro" name="robot_name">
+    <!-- 实例参数：
+         prefix            TF 帧前缀（如 robot01_），空则单机根命名空间
+         namespace         ROS 命名空间（如 robot01），空则根命名空间
+         controller_params 控制器参数文件路径（默认模板；生成脚本按规格注入几何参数）
+         调用示例：xacro amr.urdf.xacro prefix:=robot01_ namespace:=robot01
+    -->
+    <xacro:arg name="prefix" default=""/>
+    <xacro:arg name="namespace" default=""/>
+    <xacro:arg name="controller_params" default="$(find amr_description)/config/amr_ros2_controller.yaml"/>
+    <!-- 几何参数：默认值与 config/amr_v1.yaml 一致，生成脚本从规格文件覆盖传入 -->
+    <xacro:arg name="car_length" default="0.6"/>
+    <xacro:arg name="car_width" default="0.4"/>
+    <xacro:arg name="car_height" default="0.15"/>
+    <xacro:arg name="wheel_radius" default="0.064"/>
+    <xacro:arg name="wheel_length" default="0.06"/>
+    <xacro:arg name="wheel_mass" default="1.0"/>
     <!--基础部分-->
-    <xacro:include filename="$(find amr_description)/urdf/amr_description/base.urdf.xacro"/>
+    <xacro:include filename="$(find amr_description)/urdf/base.urdf.xacro"/>
     <!--传感器部分-->
-    <xacro:include filename="$(find amr_description)/urdf/amr_description/sensor/imu.urdf.xacro"/>
-    <xacro:include filename="$(find amr_description)/urdf/amr_description/sensor/camera.urdf.xacro"/>
-    <xacro:include filename="$(find amr_description)/urdf/amr_description/sensor/laser.urdf.xacro"/>
+    <xacro:include filename="$(find amr_description)/urdf/sensor/imu.urdf.xacro"/>
+    <xacro:include filename="$(find amr_description)/urdf/sensor/camera.urdf.xacro"/>
+    <xacro:include filename="$(find amr_description)/urdf/sensor/laser.urdf.xacro"/>
     <!--执行器部分-->
-    <xacro:include filename="$(find amr_description)/urdf/amr_description/actuator/wheel.urdf.xacro"/>
-    <xacro:include filename="$(find amr_description)/urdf/amr_description/actuator/caster.urdf.xacro"/>
+    <xacro:include filename="$(find amr_description)/urdf/actuator/wheel.urdf.xacro"/>
+    <xacro:include filename="$(find amr_description)/urdf/actuator/caster.urdf.xacro"/>
     <!--插件部分-->
-    <!-- <xacro:include filename="$(find amr_description)/urdf/amr_description/plugins/gazebo_control_plugin.xacro"/> -->
-    <xacro:include filename="$(find amr_description)/urdf/amr_description/plugins/gazebo_sensor_plugin.xacro"/>
-    <xacro:include filename="$(find amr_description)/urdf/amr_description/amr.ros2_control.xacro"/>
+    <!-- <xacro:include filename="$(find amr_description)/urdf/plugins/gazebo_control_plugin.xacro"/> -->
+    <xacro:include filename="$(find amr_description)/urdf/plugins/gazebo_sensor_plugin.xacro"/>
+    <xacro:include filename="$(find amr_description)/urdf/amr.ros2_control.xacro"/>
     <!-- PI 值 -->
     <xacro:property name="PI" value="3.1415927"/>
-    <!-- 底盘尺寸 -->
-    <xacro:property name="car_length" value="0.6"/>
-    <xacro:property name="car_width" value="0.4"/>
-    <xacro:property name="car_height" value="0.15"/>
-    <!-- 轮胎尺寸 -->
-    <xacro:property name="wheel_radius" value="0.064"/>
-    <xacro:property name="wheel_length" value="0.06"/>
-    <!-- 轮胎关节平移量 -->
+    <!-- 轮胎关节平移量（由几何参数推导，勿手改） -->
     <xacro:property name="wheel_joint_y" value="${car_width / 2 - wheel_length / 2 - 0.01}"/>
     <xacro:property name="wheel_joint_z" value="${-car_height / 2}"/>
@@ -40,17 +49,17 @@
     </material>
     <!-- 调用底盘，统一使用全局尺寸 -->
-    <xacro:base_xacro length="${car_length}" width="${car_width}" height="${car_height}" wheel_radius="${wheel_radius}"/>
+    <xacro:base_xacro length="${car_length}" width="${car_width}" height="${car_height}" wheel_radius="${wheel_radius}" prefix="${prefix}"/>
     <!-- 调用传感器模块 -->
-    <xacro:imu_xacro imu_name="imu" length="0.02" width="0.02" height="0.02" xyz="0 0 0.02"/>
-    <xacro:camera_xacro length="0.02" width="0.1" height="0.02" xyz="${car_length / 2 - 0.01} 0 ${car_height / 2}"/>
-    <xacro:laser_xacro radius="0.02" length="0.02" xyz="0 0 0.1"/>
+    <xacro:imu_xacro imu_name="imu" length="0.02" width="0.02" height="0.02" xyz="0 0 0.02" prefix="${prefix}"/>
+    <xacro:camera_xacro length="0.02" width="0.1" height="0.02" xyz="${car_length / 2 - 0.01} 0 ${car_height / 2}" prefix="${prefix}"/>
+    <xacro:laser_xacro radius="0.02" length="0.02" xyz="0 0 0.1" prefix="${prefix}"/>
     <!-- 调用执行器模块 -->
-    <xacro:wheel_xacro wheel_name="left" radius="${wheel_radius}" length="${wheel_length}" xyz="0 ${wheel_joint_y} ${wheel_joint_z}"/>
-    <xacro:wheel_xacro wheel_name="right" radius="${wheel_radius}" length="${wheel_length}" xyz="0 ${-wheel_joint_y} ${wheel_joint_z}"/>
-    <xacro:caster_xacro caster_name="front" radius="${wheel_radius}" xyz="${car_length / 2 - wheel_radius - 0.02} 0 ${wheel_joint_z}"/>
-    <xacro:caster_xacro caster_name="back" radius="${wheel_radius}" xyz="${-(car_length / 2 - wheel_radius - 0.02)} 0 ${wheel_joint_z}"/>
+    <xacro:wheel_xacro wheel_name="left" radius="${wheel_radius}" length="${wheel_length}" xyz="0 ${wheel_joint_y} ${wheel_joint_z}" prefix="${prefix}" mass="${wheel_mass}"/>
+    <xacro:wheel_xacro wheel_name="right" radius="${wheel_radius}" length="${wheel_length}" xyz="0 ${-wheel_joint_y} ${wheel_joint_z}" prefix="${prefix}" mass="${wheel_mass}"/>
+    <xacro:caster_xacro caster_name="front" radius="${wheel_radius}" xyz="${car_length / 2 - wheel_radius - 0.02} 0 ${wheel_joint_z}" prefix="${prefix}"/>
+    <xacro:caster_xacro caster_name="back" radius="${wheel_radius}" xyz="${-(car_length / 2 - wheel_radius - 0.02)} 0 ${wheel_joint_z}" prefix="${prefix}"/>
     <!-- 调用插件模块 -->
-    <!-- <xacro:gazebo_control_plugin left_joint_name="left_wheel_joint" right_joint_name="right_wheel_joint" wheel_separation="${wheel_joint_y * 2}" wheel_diameter="${wheel_radius * 2}"/> -->
-    <xacro:gazebo_sensor_plugin/>
-    <xacro:amr_ros2_control left_joint_name="left_wheel_joint" right_joint_name="right_wheel_joint"/>
+    <!-- <xacro:gazebo_control_plugin left_joint_name="${prefix}left_wheel_joint" right_joint_name="${prefix}right_wheel_joint" wheel_separation="${wheel_joint_y * 2}" wheel_diameter="${wheel_radius * 2}" base_frame="${prefix}base_footprint" namespace="${namespace}"/> -->
+    <xacro:gazebo_sensor_plugin prefix="${prefix}" namespace="${namespace}"/>
+    <xacro:amr_ros2_control left_joint_name="${prefix}left_wheel_joint" right_joint_name="${prefix}right_wheel_joint" prefix="${prefix}" namespace="${namespace}" controller_params="${controller_params}"/>
 </robot>

File: robot_ws/src/amr_description/urdf/base.urdf.xacro (robot description, xacro)
@@ -1,9 +1,9 @@
 <?xml version="1.0"?>
 <robot xmlns:xacro="http://www.ros.org/wiki/xacro">
-    <xacro:include filename="$(find amr_description)/urdf/amr_description/common_inertia.xacro"/>
+    <xacro:include filename="$(find amr_description)/urdf/common_inertia.xacro"/>
     <!-- 声明 base 模块 -->
-    <xacro:macro name="base_xacro" params="length width height wheel_radius">
-        <link name="base_footprint"/>
-        <link name="base_link">
+    <xacro:macro name="base_xacro" params="length width height wheel_radius prefix">
+        <link name="${prefix}base_footprint"/>
+        <link name="${prefix}base_link">
             <visual>
                 <geometry>
@@ -22,10 +22,10 @@
             <xacro:box_inertia m="${20.0}" l="${length}" w="${width}" h="${height}"/>
         </link>
-        <joint name="base_link_joint" type="fixed">
-            <parent link="base_footprint"/>
-            <child link="base_link"/>
+        <joint name="${prefix}base_link_joint" type="fixed">
+            <parent link="${prefix}base_footprint"/>
+            <child link="${prefix}base_link"/>
             <origin xyz="0.0 0.0 ${height / 2 + wheel_radius - 0.001}"/>
         </joint>
-        <gazebo reference="base_link">
+        <gazebo reference="${prefix}base_link">
             <material>Gazebo/Orange</material>
         </gazebo>

File: robot_ws/src/amr_description/urdf/plugins/gazebo_sensor_plugin.xacro (robot description, xacro)
@@ -1,14 +1,15 @@
 <?xml version="1.0"?>
 <robot xmlns:xacro="http://www.ros.org/wiki/xacro">
-    <xacro:macro name="gazebo_sensor_plugin">
-        <gazebo reference="laser_link">
+    <!-- prefix：TF 帧前缀（如 robot01_）；namespace：传感器话题命名空间（如 robot01，空为根） -->
+    <xacro:macro name="gazebo_sensor_plugin" params="prefix namespace">
+        <gazebo reference="${prefix}laser_link">
             <sensor name="laserscan" type="ray">
                 <plugin name="laserscan" filename="libgazebo_ros_ray_sensor.so">
                     <ros>
-                        <namespace>/</namespace>
+                        <namespace>${namespace}</namespace>
                         <remapping>~/out:=scan</remapping>
                     </ros>
                     <output_type>sensor_msgs/LaserScan</output_type>
-                    <frame_name>laser_link</frame_name>
+                    <frame_name>${prefix}laser_link</frame_name>
                 </plugin>
                 <always_on>true</always_on>
@@ -42,9 +43,9 @@
             </sensor>
         </gazebo>
-        <gazebo reference="imu_link">
+        <gazebo reference="${prefix}imu_link">
             <sensor name="imu_sensor" type="imu">
                 <plugin name="imu_plugin" filename="libgazebo_ros_imu_sensor.so">
                     <ros>
-                        <namespace>/</namespace>
+                        <namespace>${namespace}</namespace>
                         <remapping>~/out:=imu</remapping>
                     </ros>
@@ -110,8 +111,11 @@
             </sensor>
         </gazebo>
-        <gazebo reference="camera_link">
+        <gazebo reference="${prefix}camera_link">
             <sensor type="depth" name="camera_sensor">
                 <plugin name="depth_camera" filename="libgazebo_ros_camera.so">
-                    <frame_name>camera_optical_link</frame_name>
+                    <ros>
+                        <namespace>${namespace}</namespace>
+                    </ros>
+                    <frame_name>${prefix}camera_optical_link</frame_name>
                 </plugin>
                 <always_on>true</always_on>

File: robot_ws/src/amr_description/urdf/sensor/camera.urdf.xacro (robot description, xacro)
@@ -1,7 +1,7 @@
 <?xml version="1.0"?>
 <robot xmlns:xacro="http://www.ros.org/wiki/xacro">
-    <xacro:include filename="$(find amr_description)/urdf/amr_description/common_inertia.xacro"/>
-    <xacro:macro name="camera_xacro" params="length width height xyz">
-        <link name="camera_link">
+    <xacro:include filename="$(find amr_description)/urdf/common_inertia.xacro"/>
+    <xacro:macro name="camera_xacro" params="length width height xyz prefix">
+        <link name="${prefix}camera_link">
             <visual>
                 <geometry>
@@ -22,13 +22,13 @@
              <xacro:box_inertia m="${0.6}" l="${length}" w="${width}" h="${height}"/>
         </link>
-        <joint name="camera_joint" type="fixed">
-            <parent link="base_link"/>
-            <child link="camera_link"/>
+        <joint name="${prefix}camera_joint" type="fixed">
+            <parent link="${prefix}base_link"/>
+            <child link="${prefix}camera_link"/>
             <origin xyz="${xyz}"/>
         </joint>
-        <link name="camera_optical_link"></link>
-        <joint name="camera_optical_joint" type="fixed">
-            <parent link="camera_link"/>
-            <child link="camera_optical_link"/>
+        <link name="${prefix}camera_optical_link"></link>
+        <joint name="${prefix}camera_optical_joint" type="fixed">
+            <parent link="${prefix}camera_link"/>
+            <child link="${prefix}camera_optical_link"/>
             <origin xyz="0 0 0" rpy="${-PI / 2} 0.0 ${-PI / 2} "/>
         </joint>

File: robot_ws/src/amr_description/urdf/sensor/imu.urdf.xacro (robot description, xacro)
@@ -1,8 +1,8 @@
 <?xml version="1.0"?>
 <robot xmlns:xacro="http://www.ros.org/wiki/xacro">
-    <xacro:include filename="$(find amr_description)/urdf/amr_description/common_inertia.xacro"/>
+    <xacro:include filename="$(find amr_description)/urdf/common_inertia.xacro"/>
     <!-- 声明 IMU 模块 -->
-    <xacro:macro name="imu_xacro" params="imu_name length width height xyz">
-        <link name="${imu_name}_link">
+    <xacro:macro name="imu_xacro" params="imu_name length width height xyz prefix">
+        <link name="${prefix}${imu_name}_link">
             <visual>
                 <geometry>
@@ -21,7 +21,7 @@
              <xacro:box_inertia m="${1.0}" l="${length}" w="${width}" h="${height}"/>
         </link>
-        <joint name="${imu_name}_joint" type="fixed">
-            <parent link="base_link"/>
-            <child link="${imu_name}_link"/>
+        <joint name="${prefix}${imu_name}_joint" type="fixed">
+            <parent link="${prefix}base_link"/>
+            <child link="${prefix}${imu_name}_link"/>
             <origin xyz="${xyz}" rpy="0.0 0.0 0.0"/>
         </joint>

File: robot_ws/src/amr_description/urdf/sensor/laser.urdf.xacro (robot description, xacro)
@@ -1,7 +1,7 @@
 <?xml version="1.0"?>
 <robot xmlns:xacro="http://www.ros.org/wiki/xacro">
-    <xacro:include filename="$(find amr_description)/urdf/amr_description/common_inertia.xacro"/>
-    <xacro:macro name="laser_xacro" params="radius length xyz">
-        <link name="laser_cylinder_link">
+    <xacro:include filename="$(find amr_description)/urdf/common_inertia.xacro"/>
+    <xacro:macro name="laser_xacro" params="radius length xyz prefix">
+        <link name="${prefix}laser_cylinder_link">
             <visual>
                 <geometry>
@@ -22,10 +22,10 @@
             <xacro:cylinder_inertia m="${0.1}" r="0.01" h="0.1"/>
         </link>
-        <joint name="claser_cylinder_joint" type="fixed">
-            <parent link="base_link"/>
-            <child link="laser_cylinder_link"/>
+        <joint name="${prefix}claser_cylinder_joint" type="fixed">
+            <parent link="${prefix}base_link"/>
+            <child link="${prefix}laser_cylinder_link"/>
             <origin xyz="${xyz}"/>
         </joint>
-        <link name="laser_link">
+        <link name="${prefix}laser_link">
             <visual>
                 <geometry>
@@ -46,13 +46,13 @@
             <xacro:cylinder_inertia m="${0.2}" r="${radius}" h="${length}"/>
         </link>
-        <joint name="laser_joint" type="fixed">
-            <parent link="laser_cylinder_link"/>
-            <child link="laser_link"/>
+        <joint name="${prefix}laser_joint" type="fixed">
+            <parent link="${prefix}laser_cylinder_link"/>
+            <child link="${prefix}laser_link"/>
             <origin xyz="0 0 0.05"/>
         </joint>
-        <gazebo reference="laser_cylinder_link">
+        <gazebo reference="${prefix}laser_cylinder_link">
             <material>Gazebo/Black</material>
         </gazebo>
-        <gazebo reference="laser_link">
+        <gazebo reference="${prefix}laser_link">
             <material>Gazebo/Black</material>
         </gazebo>
