Commit message: fixed amr_description

File: robot_ws/src/amr_description/urdf/amr.ros2_control.xacro (robot description, xacro)
@@ -9,5 +9,5 @@
     -->
     <xacro:macro name="amr_ros2_control" params="left_joint_name right_joint_name prefix namespace controller_params">
-        <ros2_control name="AmrRobotGazeboSystem" type="system">
+        <ros2_control name="${prefix}AmrRobotGazeboSystem" type="system">
                 <hardware>
                     <plugin>gazebo_ros2_control/GazeboSystem</plugin>
@@ -17,8 +17,4 @@
                         <param name="min">-1</param>
                         <param name="max">1</param>
-                    </command_interface>
-                    <command_interface name="effort">
-                        <param name="min">-0.1</param>
-                        <param name="max">0.1</param>
                     </command_interface>
                     <state_interface name="position" />
@@ -31,8 +27,4 @@
                         <param name="max">1</param>
                     </command_interface>
-                    <command_interface name="effort">
-                        <param name="min">-0.1</param>
-                        <param name="max">0.1</param>
-                    </command_interface>
                     <state_interface name="position" />
                     <state_interface name="velocity" />
@@ -41,8 +33,8 @@
         </ros2_control>
         <gazebo>
-            <plugin filename="libgazebo_ros2_control.so" name="gazebo_ros2_control">
+            <plugin filename="libgazebo_ros2_control.so" name="${prefix}gazebo_ros2_control">
                 <parameters>${controller_params}</parameters>
                 <ros>
-                    <namespace>${namespace}</namespace>
+                    <namespace>/${namespace}</namespace>
                     <remapping>amr_diff_drive_controller/cmd_vel_unstamped:=cmd_vel</remapping>
                     <remapping>amr_diff_drive_controller/odom:=odom</remapping>

File: robot_ws/src/amr_description/urdf/amr.urdf.xacro (robot description, xacro)
@@ -17,4 +17,14 @@
     <xacro:arg name="wheel_length" default="0.06"/>
     <xacro:arg name="wheel_mass" default="1.0"/>
+    <!-- 将 xacro arg 转换成 property，供后续表达式使用 -->
+    <xacro:property name="prefix" value="$(arg prefix)"/>
+    <xacro:property name="namespace" value="$(arg namespace)"/>
+    <xacro:property name="controller_params" value="$(arg controller_params)"/>
+    <xacro:property name="car_length" value="$(arg car_length)"/>
+    <xacro:property name="car_width" value="$(arg car_width)"/>
+    <xacro:property name="car_height" value="$(arg car_height)"/>
+    <xacro:property name="wheel_radius" value="$(arg wheel_radius)"/>
+    <xacro:property name="wheel_length" value="$(arg wheel_length)"/>
+    <xacro:property name="wheel_mass" value="$(arg wheel_mass)"/>
     <!--基础部分-->
     <xacro:include filename="$(find amr_description)/urdf/base.urdf.xacro"/>

File: robot_ws/src/amr_description/urdf/plugins/gazebo_control_plugin.xacro (robot description, xacro)
@@ -21,5 +21,5 @@
             <plugin name='diff_drive' filename='libgazebo_ros_diff_drive.so'>
                 <ros>
-                    <namespace>${namespace}</namespace>
+                    <namespace>/${namespace}</namespace>
                     <remapping>cmd_vel:=cmd_vel</remapping>
                     <remapping>odom:=odom</remapping>

File: robot_ws/src/amr_description/urdf/plugins/gazebo_sensor_plugin.xacro (robot description, xacro)
@@ -7,5 +7,5 @@
                 <plugin name="laserscan" filename="libgazebo_ros_ray_sensor.so">
                     <ros>
-                        <namespace>${namespace}</namespace>
+                        <namespace>/${namespace}</namespace>
                         <remapping>~/out:=scan</remapping>
                     </ros>
@@ -47,5 +47,5 @@
                 <plugin name="imu_plugin" filename="libgazebo_ros_imu_sensor.so">
                     <ros>
-                        <namespace>${namespace}</namespace>
+                        <namespace>/${namespace}</namespace>
                         <remapping>~/out:=imu</remapping>
                     </ros>
@@ -115,5 +115,5 @@
                 <plugin name="depth_camera" filename="libgazebo_ros_camera.so">
                     <ros>
-                        <namespace>${namespace}</namespace>
+                        <namespace>/${namespace}</namespace>
                     </ros>
                     <frame_name>${prefix}camera_optical_link</frame_name>
